File: hardware/Low Pass Gate.brd (EAGLE design)
At the start: 40.6 x 100 mm, 87 parts, among them IC2 LM397, IC5 LM397, P1 POWER_SIMPLE10_SHROUDED, U1 OPAMP-QUADSO14, U2 OPAMP-QUADSO14

Commit message: fix C4/C13 value (that was resulting in 5.6x f(c) in filter)
Parts:
- C13, C4: value 100p -> 560p
Changed lines of the file:
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@@
 <attribute name="VALUE" x="20.7645" y="31.0515" size="0.4064" layer="27" font="vector" ratio="13" rot="R90" align="center-left"/>
 </element>
-<element name="C13" library="SparkFun-Passives" package="0805" value="100p" x="20.955" y="13.335" smashed="yes" rot="R90">
+<element name="C13" library="SparkFun-Passives" package="0805" value="560p" x="20.955" y="13.335" smashed="yes" rot="R90">
 <attribute name="NAME" x="20.955" y="15.113" size="0.5588" layer="25" font="vector" ratio="13" rot="R90" align="center-left"/>
 <attribute name="VALUE" x="21.717" y="15.1765" size="0.4064" layer="27" font="vector" ratio="10" rot="R90" align="center-left"/>
@@
 <attribute name="OC_NEWARK" value="95F9033" x="19.05" y="72.39" size="1.778" layer="28" rot="MR270" display="off"/>
 </element>
-<element name="C4" library="SparkFun-Passives" package="0805" value="100p" x="20.955" y="64.135" smashed="yes" rot="R90">
+<element name="C4" library="SparkFun-Passives" package="0805" value="560p" x="20.955" y="64.135" smashed="yes" rot="R90">
 <attribute name="NAME" x="20.7645" y="65.913" size="0.5588" layer="25" font="vector" ratio="13" rot="R90" align="center-left"/>
 <attribute name="VALUE" x="21.717" y="65.9765" size="0.4064" layer="27" font="vector" ratio="13" rot="R90"/>

Commit message: Additional fix for C4/C13 value causing audio bleedthrough at low mute settings
Parts:
- C13, C4: value 560p -> 1500p
Changed lines of the file:
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@@
 <attribute name="VALUE" x="20.7645" y="31.0515" size="0.4064" layer="27" font="vector" ratio="13" rot="R90" align="center-left"/>
 </element>
-<element name="C13" library="SparkFun-Passives" package="0805" value="560p" x="20.955" y="13.335" smashed="yes" rot="R90">
+<element name="C13" library="SparkFun-Passives" package="0805" value="1500p" x="20.955" y="13.335" smashed="yes" rot="R90">
 <attribute name="NAME" x="20.955" y="15.113" size="0.5588" layer="25" font="vector" ratio="13" rot="R90" align="center-left"/>
 <attribute name="VALUE" x="21.717" y="15.1765" size="0.4064" layer="27" font="vector" ratio="10" rot="R90" align="center-left"/>
@@
 <attribute name="OC_NEWARK" value="95F9033" x="19.05" y="72.39" size="1.778" layer="28" rot="MR270" display="off"/>
 </element>
-<element name="C4" library="SparkFun-Passives" package="0805" value="560p" x="20.955" y="64.135" smashed="yes" rot="R90">
+<element name="C4" library="SparkFun-Passives" package="0805" value="1500p" x="20.955" y="64.135" smashed="yes" rot="R90">
 <attribute name="NAME" x="20.7645" y="65.913" size="0.5588" layer="25" font="vector" ratio="13" rot="R90" align="center-left"/>
 <attribute name="VALUE" x="21.717" y="65.9765" size="0.4064" layer="27" font="vector" ratio="13" rot="R90"/>
