File: hardware/Low Pass Gate.brd (EAGLE design)
At the start: 40.6 x 100 mm, 87 parts, among them IC2 LM397, IC5 LM397, P1 POWER_SIMPLE10_SHROUDED, U1 OPAMP-QUADSO14, U2 OPAMP-QUADSO14

Commit message: adjust led drive current resistor
Parts:
- R27, R9: value 1K -> 2K2
Changed lines of the file:
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@@
 <attribute name="VALUE" x="23.876" y="65.913" size="0.4064" layer="27" font="vector" ratio="13" rot="R90"/>
 </element>
-<element name="R9" library="SparkFun-Passives" package="0603-RES" value="1K" x="24.765" y="64.135" smashed="yes" rot="R270">
+<element name="R9" library="SparkFun-Passives" package="0603-RES" value="2K2" x="24.765" y="64.135" smashed="yes" rot="R270">
 <attribute name="NAME" x="24.8285" y="65.913" size="0.5588" layer="25" font="vector" ratio="13" rot="R90" align="center-left"/>
 <attribute name="VALUE" x="25.781" y="65.913" size="0.4064" layer="27" font="vector" ratio="13" rot="R90"/>
 </element>
-<element name="R27" library="SparkFun-Passives" package="0603-RES" value="1K" x="24.765" y="13.335" smashed="yes" rot="R270">
+<element name="R27" library="SparkFun-Passives" package="0603-RES" value="2K2" x="24.765" y="13.335" smashed="yes" rot="R270">
 <attribute name="NAME" x="24.8285" y="15.113" size="0.5588" layer="25" font="vector" ratio="13" rot="R90" align="center-left"/>
 <attribute name="VALUE" x="25.781" y="15.113" size="0.4064" layer="27" font="vector" ratio="13" rot="R90"/>

Commit message: fix drive resistor value
Parts:
- R27, R9: value 2K2 -> 4K7
Changed lines of the file:
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@@
 <attribute name="VALUE" x="23.876" y="65.913" size="0.4064" layer="27" font="vector" ratio="13" rot="R90"/>
 </element>
-<element name="R9" library="SparkFun-Passives" package="0603-RES" value="2K2" x="24.765" y="64.135" smashed="yes" rot="R270">
+<element name="R9" library="SparkFun-Passives" package="0603-RES" value="4K7" x="24.765" y="64.135" smashed="yes" rot="R270">
 <attribute name="NAME" x="24.8285" y="65.913" size="0.5588" layer="25" font="vector" ratio="13" rot="R90" align="center-left"/>
 <attribute name="VALUE" x="25.781" y="65.913" size="0.4064" layer="27" font="vector" ratio="13" rot="R90"/>
 </element>
-<element name="R27" library="SparkFun-Passives" package="0603-RES" value="2K2" x="24.765" y="13.335" smashed="yes" rot="R270">
+<element name="R27" library="SparkFun-Passives" package="0603-RES" value="4K7" x="24.765" y="13.335" smashed="yes" rot="R270">
 <attribute name="NAME" x="24.8285" y="15.113" size="0.5588" layer="25" font="vector" ratio="13" rot="R90" align="center-left"/>
 <attribute name="VALUE" x="25.781" y="15.113" size="0.4064" layer="27" font="vector" ratio="13" rot="R90"/>
